Commit message: add tarea 1 related files

File: brazos/scara_fcfm_model/scara.urdf (robot description, URDF)
Before this commit: robot scara, 4 links, 3 joints
Links:
- link zeta: geometry visual mesh filename=package://scara_fcfm_model/meshes/z_corrected.dae

File: efectores/scara/tweezer/tweezer.urdf (robot description, URDF)
Before this commit: robot scara_tweezer, 3 links, 2 joints
Links:
- added link invisible_link, mass 0.001; collision mesh filename=package://tweezer/meshes/visual/scara_twbase.stl; visual mesh filename=package://tweezer/meshes/visual/scara_twbase.stl
- link base_link: mass 0.01 -> None; geometry visual mesh filename=package://tweezer/meshes/visual/scara_twbase.stl
Joints:
- added joint rotacion_gripper: type revolute, parent base_link, child invisible_link, origin xyz=0 0 0, axis 0 0 1, limit lower=-1.57 upper=1.57 effort=35 velocity=8
- joint joint1: axis 1 0 0 -> 0 1 0; limit lower=-0.03 upper=0 effort=10 velocity=10 -> lower=-0.03 upper=0 effort=10 velocity=1; parent base_link -> invisible_link
- joint joint2: axis 1 0 0 -> 0 1 0; limit lower=0 upper=0.03 effort=10 velocity=10 -> lower=0 upper=0.03 effort=10 velocity=1; parent base_link -> invisible_link
