Commit message: fix scara call

File: modelos/manipuladores/scara/scara.urdf (robot description, URDF)
Before this commit: robot scara, 4 links, 3 joints
Links:
- link base_link: geometry collision mesh filename=package://scara/meshes/base_corrected.dae; visual mesh filename=package://scara/meshes/base_corrected.dae
- link humero: geometry collision mesh filename=package://scara/meshes/humero_corrected.dae; visual mesh filename=package://scara/meshes/humero_corrected.dae
- link rc: geometry collision mesh filename=package://scara/meshes/rc_corrected.dae; visual mesh filename=package://scara/meshes/rc_corrected.dae
- link zeta: geometry visual mesh filename=package://scara/meshes/z_corrected.dae
