Commit message: update urdf

File: modelos/efectores/puntero/puntero.urdf (robot description, URDF)
Before this commit: robot puntero, 1 links, 0 joints
Links:
- link baseLink: geometry collision mesh filename=package://puntero/meshes/collision/puntero.stl; visual mesh filename=package://puntero/meshes/visual/puntero.stl

File: modelos/manipuladores/kuka/kr6_2.urdf (robot description, URDF)
Before this commit: robot kuka-model, 7 links, 6 joints
Links:
- link base: geometry collision mesh filename=package://kuka/meshes/collision/base_link.stl; visual mesh filename=package://kuka/meshes/visual/base_link.stl
- link link_1: geometry collision mesh filename=package://kuka/meshes/collision/link_1.stl; visual mesh filename=package://kuka/meshes/visual/link_1.stl
- link link_2: geometry collision mesh filename=package://kuka/meshes/collision/link_2.stl; visual mesh filename=package://kuka/meshes/visual/link_2.stl
- link link_3: geometry collision mesh filename=package://kuka/meshes/collision/link_3.stl; visual mesh filename=package://kuka/meshes/visual/link_3.stl
- link link_4: geometry collision mesh filename=package://kuka/meshes/collision/link_4.stl; visual mesh filename=package://kuka/meshes/visual/link_4.stl
- link link_5: geometry collision mesh filename=package://kuka/meshes/collision/link_5.stl; visual mesh filename=package://kuka/meshes/visual/link_5.stl
- link link_6: geometry collision mesh filename=package://kuka/meshes/collision/link_6.stl; visual mesh filename=package://kuka/meshes/visual/link_6.stl
