Commit message: Se incorporan las collision en ruedas y cambio de joints

File: modelos/base_movil/omnibase.urdf (robot description, URDF)
Before this commit: robot base_link_only, 10 links, 9 joints
Links:
- removed link world
- link wheel_1: geometry collision mesh filename=ME5150_tutorials\modelos\base_movil\meshes\cilindro_ruedas_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; visual mesh filename=ME5150_tutorials\modelos\base_movil\meshes\ruedader.stl
- link wheel_2: geometry collision mesh filename=ME5150_tutorials\modelos\base_movil\meshes\cilindro_ruedas_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; visual mesh filename=ME5150_tutorials\modelos\base_movil\meshes\ruedaizq.stl
- link wheel_3: geometry collision mesh filename=ME5150_tutorials\modelos\base_movil\meshes\cilindro_ruedas_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; visual mesh filename=ME5150_tutorials\modelos\base_movil\meshes\ruedaizq.stl
- link wheel_4: geometry collision mesh filename=ME5150_tutorials\modelos\base_movil\meshes\cilindro_ruedas_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; visual mesh filename=ME5150_tutorials\modelos\base_movil\meshes\ruedader.stl
Joints:
- removed joint fixed_joint
- joint rueda1: limit lower=-3.1416 upper=3.1416 effort=100 velocity=3.14 -> (none); type revolute -> continuous
- joint rueda2: limit lower=-3.1416 upper=3.1416 effort=100 velocity=3.14 -> (none); type revolute -> continuous
- joint rueda3: limit lower=-3.1416 upper=3.1416 effort=100 velocity=3.14 -> (none); type revolute -> continuous
- joint rueda4: limit lower=-3.1416 upper=3.1416 effort=100 velocity=3.14 -> (none); type revolute -> continuous

Commit message: edit collision orientation and rotation axis for each wheel

File: modelos/base_movil/omnibase.urdf (robot description, URDF)
Before this commit: robot base_link_only, 9 links, 8 joints
Joints:
- joint rueda1: axis 0 0 1 -> 0 1 0
- joint rueda2: axis 0 0 1 -> 0 1 0
- joint rueda3: axis 0 0 1 -> 0 1 0
- joint rueda4: axis 0 0 1 -> 0 1 0

Commit message: Position and orientation of the wheels fixed

File: modelos/base_movil/omnibase.urdf (robot description, URDF)
Before this commit: robot base_link_only, 9 links, 8 joints
Joints:
- joint motor_dc_1_joint: origin xyz=0.06425 0.041487 0.0 rpy=0.0 0.0 0.0 -> xyz=0.06425 0.043487 -0.01287 rpy=-1.5708 0.0 3.14
- joint motor_dc_2_joint: origin xyz=0.06425 -0.041487 0.0 rpy=0.0 0.0 0.0 -> xyz=0.06425 -0.043487 -0.01287 rpy=1.5708 0.0 3.14
- joint motor_dc_3_joint: origin xyz=-0.06425 0.041487 0.0 rpy=0.0 0.0 0.0 -> xyz=-0.06425 0.043487 -0.01287 rpy=1.5708 0.0 0.0
- joint motor_dc_4_joint: origin xyz=-0.06425 -0.041487 0.0 rpy=0.0 0.0 0.0 -> xyz=-0.06425 -0.043487 -0.01287 rpy=-1.5708 0.0 0.0
- joint rueda1: axis 0 1 0 -> 0 0 1; origin xyz=0.0 0.025 0.0 -> xyz=0.0 0.0 -0.027043 rpy=0 3.14 0
- joint rueda2: axis 0 1 0 -> 0 0 1; origin xyz=0.0 -0.025 0.0 -> xyz=0.0 0.0 -0.027043 rpy=0 -3.14 0
- joint rueda3: axis 0 1 0 -> 0 0 1; origin xyz=0.0 0.025 0.0 -> xyz=0.0 0.0 -0.027043 rpy=-3.14 0 0
- joint rueda4: axis 0 1 0 -> 0 0 1; origin xyz=0.0 -0.025 0.0 -> xyz=0.0 0.0 -0.027043 rpy=3.14 0 0
