Commit message: Added a robotic arm folder

File: modelos/manipuladores/ejemplo_brazo/roboticarm/roboticarm.urdf (robot description, URDF)
Before this commit: robot robotic_arm, 4 links, 3 joints
Links:
- link arm_link1: mass 1297 -> 1; geometry collision mesh filename=modelos/manipuladores/ejemplo_brazo/roboticarm/meshes/prime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; visual mesh filename=modelos/manipuladores/ejemplo_brazo/roboticarm/meshes/prime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
- link arm_link2: mass 8747 -> 9; geometry collision mesh filename=modelos/manipuladores/ejemplo_brazo/roboticarm/meshes/segun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; visual mesh filename=modelos/manipuladores/ejemplo_brazo/roboticarm/meshes/segun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
- link base_link: mass 3815 -> 4; geometry collision mesh filename=modelos/manipuladores/ejemplo_brazo/roboticarm/meshes/base_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; visual mesh filename=modelos/manipuladores/ejemplo_brazo/roboticarm/meshes/base_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
- link gripper_link: mass 38.479 -> 0.04; geometry collision mesh filename=modelos/manipuladores/ejemplo_brazo/roboticarm/meshes/gripp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; visual mesh filename=modelos/manipuladores/ejemplo_brazo/roboticarm/meshes/gripp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
Joints:
- joint arm1_to_arm2: axis 0 1 0 -> 0 0 1; limit lower=-3.1416 upper=3.1416 -> lower=-1.5708 upper=1.5708; origin xyz=1.294 -0.125 1.84 rpy=0 0 0 -> xyz=1.294 0 1.84 rpy=1.5708 0 0
- joint arm2_to_gripper: axis 1 0 0 -> 0 0 1; origin xyz=1.85 0 -0.125 rpy=0 0 0 -> xyz=1.85 0 0 rpy=0 1.5708 0
