Commit message: clean repo

File: modelos/manipuladores/twolinks/twolinks.urdf (robot description, URDF)
Before this commit: robot roboticarm, 4 links, 3 joints
Links:
- link arm_link1: geometry collision mesh filename=modelos/manipuladores/twolinks/meshes/primerbrazo.stl; visual mesh filename=modelos/manipuladores/twolinks/meshes/primerbrazo.stl
- link arm_link2: geometry collision mesh filename=modelos/manipuladores/twolinks/meshes/segundobrazo.stl; visual mesh filename=modelos/manipuladores/twolinks/meshes/segundobrazo.stl
- link base_link: geometry collision mesh filename=modelos/manipuladores/twolinks/meshes/base.stl; visual mesh filename=modelos/manipuladores/twolinks/meshes/base.stl
- link gripper_link: geometry collision mesh filename=modelos/manipuladores/twolinks/meshes/gripper.stl; visual mesh filename=modelos/manipuladores/twolinks/meshes/gripper.stl
Joints:
- joint base_to_arm1: limit lower=-3.1416 upper=3.1416 -> lower=0 upper=3.1416
