Commit message: add brush

File: modelos/manipuladores/scarapris/scarapris.urdf (robot description, URDF)
Before this commit: robot skaren, 5 links, 4 joints
Links:
- added link brush, mass 5; collision mesh filename=package://scarapris/meshes/visual/brush.stl; visual mesh filename=package://scarapris/meshes/visual/brush.stl
- link antebrazo: geometry collision mesh filename=package://scarapris/meshes/visual/link_2.stl; visual mesh filename=package://scarapris/meshes/visual/link_2.stl
- link base_link: geometry collision mesh filename=package://scarapris/meshes/collision/base.stl; visual mesh filename=package://scarapris/meshes/visual/base.stl
- link humero: geometry collision mesh filename=package://scarapris/meshes/visual/link_1.stl; visual mesh filename=package://scarapris/meshes/visual/link_1.stl
- link off_x: geometry collision mesh filename=package://scarapris/meshes/visual/link_3.stl; visual mesh filename=package://scarapris/meshes/visual/link_3.stl
- link pris_z: geometry collision mesh filename=package://scarapris/meshes/visual/pris_z.stl; visual mesh filename=package://scarapris/meshes/visual/pris_z.stl
Joints:
- added joint brush: type fixed, parent pris_z, child brush, origin xyz=0 0 0 rpy=0 0 0
- joint pris_z: limit lower=-0.1 upper=0 -> lower=-0.07 upper=0

Commit message: fix brush

File: modelos/manipuladores/scarapris/scarapris.urdf (robot description, URDF)
Before this commit: robot scarapris, 6 links, 5 joints
Joints:
- joint brush: origin xyz=0 0 0 rpy=0 0 0 -> xyz=0 0 -0.07 rpy=0 0 0
- joint pris_z: limit lower=-0.07 upper=0 -> lower=-0.06 upper=0; origin xyz=0 0.04 -0.05 rpy=0 0 0 -> xyz=0 0.039 -0.05 rpy=0 0 0

Commit message: start t1

File: modelos/manipuladores/scarapris/scarapris.urdf (robot description, URDF)
Before this commit: robot scarapris, 6 links, 5 joints
Links:
- added link rod, mass 5; collision mesh filename=package://scarapris/meshes/visual/link_1_rod.stl; visual mesh filename=package://scarapris/meshes/visual/link_1_rod.stl
Joints:
- added joint rodamiento: type fixed, parent humero, child rod, origin xyz=0 0 0 rpy=0 0 0

Commit message: add color to skaren

File: modelos/manipuladores/scarapris/scarapris.urdf (robot description, URDF)
Before this commit: robot scarapris, 7 links, 6 joints
Links:
- removed link rod
Joints:
- removed joint rodamiento
