Commit message: added base and gripper to katana urdf

File: modelos/manipuladores/katana/katana.urdf (robot description, URDF)
Before this commit: robot katana_300_6m180, 9 links, 8 joints
Links:
- added link katana_base_controlbox, mass 0.5; collision mesh filename=package://katana/katana/katana_internal_controlbox.stl; visual mesh filename=package://katana/katana/katana_internal_controlbox.stl
- added link katana_l_finger_link, mass 0.0251722230462; collision mesh filename=package://katana/katana/katana_gripper_l_finger.stl; visual mesh filename=package://katana/katana/katana_gripper_l_finger.stl
- added link katana_r_finger_link, mass 0.0251722230462; collision mesh filename=package://katana/katana/katana_gripper_r_finger.stl; visual mesh filename=package://katana/katana/katana_gripper_r_finger.stl
Joints:
- added joint katana_base_controlbox_joint: type fixed, parent katana_base_controlbox, child katana_base_link, origin xyz=0 0 0.07 rpy=0 0 0, axis 0 0 1, limit lower=-3.025528 upper=2.891097 effort=1.5 velocity=2.208932
- added joint katana_l_finger_joint: type revolute, parent katana_gripper_link, child katana_l_finger_link, origin xyz=0.034 0 0 rpy=3.14159 0 0, axis 0 0 1, limit lower=-0.44 upper=0.30 effort=0.5 velocity=0.718834
- added joint katana_r_finger_joint: type revolute, parent katana_gripper_link, child katana_r_finger_link, origin xyz=0.034 0 0 rpy=0 0 0, axis 0 0 1, limit lower=-0.44 upper=0.30 effort=0.5 velocity=0.718834
- joint katana_base_frame_joint: origin xyz=0 0 ${base_height} rpy=0 0 0 -> xyz=0 0 0.2015 rpy=0 0 0
- joint katana_gripper_tool_frame_joint: origin xyz=0 0 -0.1505 rpy=0 ${M_PI/2} 0 -> xyz=0 0 -0.1505 rpy=0 1.5708 0
- joint katana_motor5_wrist_roll_joint: origin xyz=0.1523 0 0 rpy=$1.5708 0 -1.5708 -> xyz=0.1523 0 0 rpy=1.5708 0 -1.5708
